Commit message: first commit

File: src/rm_gimbal_description/urdf/rm_gimbal.urdf.xacro (robot description, xacro)
@@ -20,4 +20,6 @@
   <joint name="camera_optical_joint" type="fixed">
     <origin xyz="0 0 0" rpy="${-pi/2} 0 ${-pi/2}" />
+    <!-- <origin xyz="0 0 0" rpy="${-pi/2} 0 0"/> -->
+    <!-- <origin xyz="0 0 0" rpy="${-pi/2} 0 ${-pi}"/> -->
     <parent link="camera_link" />
     <child link="camera_optical_frame" />

Commit message: 完成部署

File: src/rm_gimbal_description/urdf/rm_gimbal.urdf.xacro (robot description, xacro)
@@ -6,5 +6,5 @@
   <link name="odom" />
   <link name="gimbal_link" />
-  <joint name="gimbal_joint" type="floating">
+  <joint name="gimbal_joint" type="continuous">
     <parent link="odom" />
     <child link="gimbal_link" />
